Commit message: kalman

File: src/robot_description/urdf/robot.urdf.xacro (robot description, xacro)
@@ -1,137 +1,90 @@
 <?xml version="1.0"?>
-<robot name="robot" xmlns:xacro="http://ros.org/wiki/xacro">
-    <xacro:include filename="$(find robot_description)/urdf/robot_gazebo.xacro"/>
-    <link name="base_footprint"/>
-    <link name="base_link">
-        <inertial>
-            <origin xyz="0 0 0.04" rpy="0.0 0.25 0.3" />
-            <mass value="8.2573504e-01"/>
-            <inertia ixx="2.2124416e-02" ixy="-1.2294101e-04" ixz="3.4938785e-04"
-                     iyy="2.1193702e-02" iyz="-5.0120904e-05"
-                     izz="2.0064271e-02" />
-        </inertial>
-        <visual>
-            <origin rpy="0 0 0" xyz="0 0 0"/>
-            <geometry>
-                <mesh filename="package://robot_description/meshes/base_link.STL"/>
-            </geometry>
-        </visual>
-        <collision>
-            <origin rpy="0 0 0" xyz="0 0 0"/>
-            <geometry>
-                <mesh filename="package://robot_description/meshes/base_link.STL"/>
-            </geometry>
-        </collision>
-    </link>
-    <joint name="base_joint" type="fixed">
-        <parent link="base_footprint"/>
-        <child link="base_link"/>
-        <origin rpy="0 0 0" xyz="0 0 0.033"/>
-    </joint>
-    <link name="wheel_right_link">
-        <inertial>
-            <origin xyz="0 -0.014 0" rpy="0 0 0" />
-            <mass value="0.0530086090966721" />
-            <inertia ixx="1.88176298336665E-05" ixy="-4.8444933029987E-10" ixz="1.88163708851143E-08"
-                     iyy="3.11510738647764E-05" iyz="-6.93560663069607E-11"
-                     izz="1.8801969558182E-05" />
-        </inertial>
-        <visual>
-            <origin rpy="1.57 0 0" xyz="0 0 0"/>
-            <geometry>
-                <mesh filename="package://robot_description/meshes/wheel_right_link.STL"/>
-            </geometry>
-        </visual>
-        <collision>
-            <origin xyz="0 -0.015 0" rpy="1.57 0 0"/>
-            <geometry>
-                <sphere radius="0.033"/>
-            </geometry>
-        </collision>
-    </link>
-    <joint name="wheel_right_joint" type="continuous">
-        <origin rpy="0 0 0" xyz="0 -0.07 0"/>
-        <parent link="base_link"/>
-        <child link="wheel_right_link"/>
-        <axis xyz="0 1 0"/>
-    </joint>
-    <link name="wheel_left_link">
-        <inertial>
-            <origin xyz="0 0.014 0" rpy="0 0 0" />
-            <mass value="0.0530086043217644" />
-            <inertia ixx="1.8792911368909E-05"  ixy="3.31256392204584E-10" ixz="-1.14082001662767E-08"
-                     iyy="3.11510738759073E-05" iyz="-3.60499245082192E-10"
-                     izz="1.88266886146847E-05" />
-        </inertial>
-        <visual>
-            <origin rpy="-1.57 0 0" xyz="0 0 0"/>
-            <geometry>
-                <mesh filename="package://robot_description/meshes/wheel_left_link.STL"/>
-            </geometry>
-        </visual>
-        <collision>
-            <origin xyz="0 0.015 0" rpy="1.57 0 0"/>
-            <geometry>
-                <sphere radius="0.033"/>
-            </geometry>
-        </collision>
-    </link>
-    <joint name="wheel_left_joint" type="continuous">
-        <origin rpy="0 0 0" xyz="0 0.07 0"/>
-        <parent link="base_link"/>
-        <child link="wheel_left_link"/>
-        <axis xyz="0 1 0"/>
-    </joint>
-    <link name="caster_front_link">
-        <inertial>
-            <origin xyz="3.89968128948481E-07 2.40073004698083E-07 0.00219173397061506" rpy="0 0 0" />
-            <mass value="1.44379265037903E-06" />
-            <inertia ixx="7.23075276010246E-11" ixy="-6.10956883467859E-16" ixz="2.22849693525031E-15"
-                     iyy="3.8713793085917E-11"  iyz="2.93909858781952E-15"
-                     izz="1.00967486676306E-10" />
-        </inertial>
-        <visual>
-            <origin rpy="0 0 0" xyz="0 0 0"/>
-            <geometry>
-                <mesh filename="package://robot_description/meshes/caster_front_link.STL"/>
-            </geometry>
-        </visual>
-        <collision>
-            <origin xyz="0 0 0" rpy="0 0 0"/>
-            <geometry>
-                <sphere radius="0.005"/>
-            </geometry>
-        </collision>
-    </link>
-    <joint name="caster_front_joint" type="fixed">
-        <origin rpy="0 0 0" xyz="0.0475 0 -0.0275"/>
-        <parent link="base_link"/>
-        <child link="caster_front_link"/>
-    </joint>
-    <link name="caster_rear_link">
-        <inertial>
-            <origin xyz="3.8996812895542E-07 2.40073004698083E-07 0.00219173397061509" rpy="0 0 0" />
-            <mass value="1.44379265037902E-06" />
-            <inertia ixx="7.23075276010246E-11" ixy="-6.10956872363424E-16" ixz="2.22849693527207E-15"
-                     iyy="3.87137930859167E-11" iyz="2.939098587861E-15"
-                     izz="1.00967486676306E-10" />
-        </inertial>
-        <visual>
-            <origin rpy="0 0 0" xyz="0 0 0"/>
-            <geometry>
-                <mesh filename="package://robot_description/meshes/caster_rear_link.STL"/>
-            </geometry>
-        </visual>
-        <collision>
-            <origin xyz="0 0 0" rpy="0 0 0"/>
-            <geometry>
-                <sphere radius="0.005"/>
-            </geometry>
-        </collision>
-    </link>
-    <joint name="caster_rear_joint" type="fixed">
-        <origin rpy="0 0 0" xyz="-0.0475 0 -0.0275"/>
-        <parent link="base_link"/>
-        <child link="caster_rear_link"/>
-    </joint>
+<robot name="robot" xmlns:xacro="http://www.ros.org/wiki/xacro">
+  <!-- Include Gazebo + transmissions -->
+  <xacro:include filename="$(find robot_description)/urdf/robot_gazebo.xacro"/>
+  <!-- Base -->
+  <link name="base_footprint"/>
+  <link name="base_link">
+    <inertial>
+      <origin xyz="0 0 0.04" rpy="0.0 0.25 0.3"/>
+      <mass value="0.82573504"/>
+      <inertia
+        ixx="0.022124416" ixy="-0.000122941"
+        ixz="0.000349387"
+        iyy="0.021193702" iyz="-0.0000501209"
+        izz="0.020064271"/>
+    </inertial>
+    <visual>
+      <geometry>
+        <mesh filename="package://robot_description/meshes/base_link.STL"/>
+      </geometry>
+    </visual>
+    <collision>
+      <geometry>
+        <mesh filename="package://robot_description/meshes/base_link.STL"/>
+      </geometry>
+    </collision>
+  </link>
+  <joint name="base_joint" type="fixed">
+    <parent link="base_footprint"/>
+    <child link="base_link"/>
+    <origin xyz="0 0 0.033" rpy="0 0 0"/>
+  </joint>
+  <!-- Right Wheel -->
+  <link name="wheel_right_link">
+    <inertial>
+      <mass value="0.053"/>
+      <inertia ixx="1.88e-05" iyy="3.11e-05" izz="1.88e-05"
+               ixy="0" ixz="0" iyz="0"/>
+    </inertial>
+    <visual>
+      <origin xyz="0 0 0" rpy="1.57 0 0"/>
+      <geometry>
+        <mesh filename="package://robot_description/meshes/wheel_right_link.STL"/>
+      </geometry>
+    </visual>
+    <collision>
+      <geometry>
+        <sphere radius="0.033"/>
+      </geometry>
+    </collision>
+  </link>
+  <joint name="wheel_right_joint" type="continuous">
+    <parent link="base_link"/>
+    <child link="wheel_right_link"/>
+    <origin xyz="0 -0.07 0" rpy="0 0 0"/>
+    <axis xyz="0 1 0"/>
+  </joint>
+  <!-- Left Wheel -->
+  <link name="wheel_left_link">
+    <inertial>
+      <mass value="0.053"/>
+      <inertia ixx="1.88e-05" iyy="3.11e-05" izz="1.88e-05"
+               ixy="0" ixz="0" iyz="0"/>
+    </inertial>
+    <visual>
+      <origin xyz="0 0 0" rpy="-1.57 0 0"/>
+      <geometry>
+        <mesh filename="package://robot_description/meshes/wheel_left_link.STL"/>
+      </geometry>
+    </visual>
+    <collision>
+      <geometry>
+        <sphere radius="0.033"/>
+      </geometry>
+    </collision>
+  </link>
+  <joint name="wheel_left_joint" type="continuous">
+    <parent link="base_link"/>
+    <child link="wheel_left_link"/>
+    <origin xyz="0 0.07 0" rpy="0 0 0"/>
+    <axis xyz="0 1 0"/>
+  </joint>
+  <!-- IMU -->
+  <link name="imu_link"/>
+  <joint name="imu_joint" type="fixed">
+    <parent link="base_link"/>
+    <child link="imu_link"/>
+    <origin xyz="0 0 0.07" rpy="3.14159 0 0"/>
+  </joint>
 </robot>

File: src/robot_description/urdf/robot_gazebo.xacro (robot description, xacro)
@@ -1,84 +1,48 @@
 <?xml version="1.0"?>
-<robot name="robot" xmlns:xacro="http://ros.org/wiki/xacro">
-<transmission name="wheel_left_transmission">
-  <type>transmission_interface/SimpleTransmission</type>
-  <joint name="wheel_left_joint">
-    <hardwareInterface>hardware_interface/VelocityJointInterface</hardwareInterface>
-  </joint>
-  <actuator name="wheel_left_motor">
-    <mechanicalReduction>1.0</mechanicalReduction>
-    <hardwareInterface>hardware_interface/VelocityJointInterface</hardwareInterface>
-  </actuator>
-</transmission>
-<transmission name="wheel_right_transmission">
-  <type>transmission_interface/SimpleTransmission</type>
-  <joint name="wheel_right_joint">
-    <hardwareInterface>hardware_interface/VelocityJointInterface</hardwareInterface>
-  </joint>
-  <actuator name="wheel_right_motor">
-    <mechanicalReduction>1.0</mechanicalReduction>
-    <hardwareInterface>hardware_interface/VelocityJointInterface</hardwareInterface>
-  </actuator>
-</transmission>
-<!-- EffortJointInterface → control torque
-VelocityJointInterface → control speed
-PositionJointInterface → control position -->
+<robot name="robot" xmlns:xacro="http://www.ros.org/wiki/xacro">
+  <!-- TRANSMISSIONS -->
+  <transmission name="wheel_left_transmission">
+    <type>transmission_interface/SimpleTransmission</type>
+    <joint name="wheel_left_joint">
+      <hardwareInterface>hardware_interface/VelocityJointInterface</hardwareInterface>
+    </joint>
+    <actuator name="wheel_left_motor">
+      <mechanicalReduction>1</mechanicalReduction>
+    </actuator>
+  </transmission>
+  <transmission name="wheel_right_transmission">
+    <type>transmission_interface/SimpleTransmission</type>
+    <joint name="wheel_right_joint">
+      <hardwareInterface>hardware_interface/VelocityJointInterface</hardwareInterface>
+    </joint>
+    <actuator name="wheel_right_motor">
+      <mechanicalReduction>1</mechanicalReduction>
+    </actuator>
+  </transmission>
+  <!-- Wheel friction -->
   <gazebo reference="wheel_left_link">
-    <mu1>1000000000000000.0</mu1> <!-- rolling direction friction -->
-    <mu2>1000000000000000.0</mu2> <!-- sideway direction friction -->
-    <kp>1000000000000.0</kp> <!-- damping -->
-    <kd>10.0</kd> <!-- joint stiffness -->
-    <minDepth>0.001</minDepth> <!-- contact surface penetration depth -->
-    <maxVel>0.1</maxVel> <!-- max contact surface velocity -->
-    <fdir1>1 0 0</fdir1> <!-- direction of the friction -->
+    <mu1>1.0</mu1>
+    <mu2>1.0</mu2>
   </gazebo>
   <gazebo reference="wheel_right_link">
-    <mu1>1000000000000000.0</mu1>
-    <mu2>1000000000000000.0</mu2>
-    <kp>1000000000000.0</kp>
-    <kd>10.0</kd>
-    <minDepth>0.001</minDepth>
-    <maxVel>0.1</maxVel>
-    <fdir1>1 0 0</fdir1>
+    <mu1>1.0</mu1>
+    <mu2>1.0</mu2>
   </gazebo>
-  <gazebo reference="caster_rear_link">
-    <mu1>0.1</mu1>
-    <mu2>0.1</mu2>
-    <kp>1000000.0</kp>
-    <kd>100.0</kd>
-    <minDepth>0.001</minDepth>
-    <maxVel>1.0</maxVel>
-  </gazebo>
-  <gazebo reference="caster_front_link">
-    <mu1>0.1</mu1>
-    <mu2>0.1</mu2>
-    <kp>1000000.0</kp>
-    <kd>100.0</kd>
-    <minDepth>0.001</minDepth>
-    <maxVel>1.0</maxVel>
-  </gazebo>
+  <!-- ROS Control -->
   <gazebo>
     <plugin name="gazebo_ros_control" filename="libgazebo_ros_control.so">
       <robotNamespace>/</robotNamespace>
-      <robotSimType>gazebo_ros_control/DefaultRobotHWSim</robotSimType>
-      <legacyModeNS>true</legacyModeNS>
+    </plugin>
+  </gazebo>
+  <!-- IMU Plugin -->
+  <gazebo>
+    <plugin name="imu_plugin" filename="libgazebo_ros_imu.so">
+      <alwaysOn>true</alwaysOn>
+      <bodyName>imu_link</bodyName>
+      <frameName>imu_link</frameName>
+      <topicName>imu</topicName>
+      <gaussianNoise>0.001</gaussianNoise>
+      <updateRate>500</updateRate>
     </plugin>
   </gazebo>
 </robot>
-<!-- <plugin name="gazebo_ros_control" filename="libgazebo_ros_control.so">
-Loads the Gazebo ROS Control plugin.
-This plugin is REQUIRED for:
-wheel controllers
-diff drive
-PID control
-Publishing joint states
-Chooses the hardware simulation type.
-DefaultRobotHWSim =
-✔ Basic wheel motors
-✔ No sensors
-✔ Uses URDF transmissions
-✔ Works for differential drive robots
-You can replace this with custom hardware simulation plugins for:
-humanoids
-manipulators
-complex joint actuators-->
